File: pcb/kudzu.kicad_pcb (KiCad board)
At the start: 4 copper layers, 90 x 130 mm, 118 parts, among them J1 USB_C_Receptacle_USB2.0, J2 ARM 10 Pin SWD, J3 6 Pin Tag Connect, J4 Conn_01x02, J5 Conn_01x02, J6 Conn_01x03, J7 GameBoy_LinkPort, J9 Conn_01x40_MountingPin, Q1 Q_PMOS_GSD, Q2 Q_PMOS_GSD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

Commit message: pcb: Rev 0-rc2
Change-Id: I24dc5247317789b953b5f4a603b2224101365fed
Reviewed-on: https://pigweed-review.googlesource.com/c/pigweed/kudzu/+/170855
Reviewed-by: Anthony DiGirolamo <tonymd@google.com>
Parts:
- moved R3 26.4 mm to (80.2, 152.3)
- moved R4 26.4 mm to (78.7, 152.3)
- moved JP6 6.70 mm to (87.3, 38.1)
- moved JP7 4.71 mm to (84.0, 38.1)
- moved TP15 3.58 mm to (130.7, 61.5)
- moved TP11 3.53 mm to (130.7, 63.6)
- moved C27 2.99 mm to (90.1, 155.7), turned to 45 degrees
- moved C28 2.83 mm to (89.0, 154.7), turned to 45 degrees
- moved JP1 2.43 mm to (90.7, 38.1)
- moved R17 2.20 mm to (106.5, 150.2)
- moved TP12 2.07 mm to (132.4, 62.6)
- moved TP14 2.07 mm to (132.4, 64.6)
- moved TP13 2.05 mm to (132.4, 60.5)
- moved R16 1.87 mm to (103.8, 150.2)
- moved R2 1.71 mm to (91.7, 152.1), turned to -135 degrees
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Connections:
- net /RP2040 and Debug/USB_DM renamed /RP2040 and Debug/USBD_N
- net /RP2040 and Debug/USB_DP renamed /RP2040 and Debug/USBD_P
Routing:
- net /RP2040 and Debug/USBD_N: track 6.32 -> 44.3 mm
- net /RP2040 and Debug/USBD_P: track 6.32 -> 44.3 mm
- net Net-(U2-USB_DP): track 41.9 -> 7.20 mm
- net Net-(U2-USB_DM): track 41.4 -> 7.24 mm
- net Net-(J7-SI): track 11.3 -> 23.6 mm
- net Net-(J7-SC): track 13.6 -> 23.5 mm
- net STATUS_B: track 122.6 -> 116.6 mm
- net GND: track 151.4 -> 157.3 mm
- net Net-(J7-SD): track 17.9 -> 23.7 mm
- net STATUS_R: track 117.7 -> 111.9 mm
- net STATUS_G: track 119.9 -> 114.2 mm
- net Net-(J7-SO): track 17.9 -> 23.5 mm
- net /RP2040 and Debug/SWCLK: track 29.6 -> 34.7 mm, vias 0 -> 2
- net /RP2040 and Debug/QSPI_SD3: track 16.9 -> 12.0 mm
- net DISP_SDI: track 129.6 -> 133.8 mm
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
Commit message: pcb: Rev 0 ready for fab!
Change-Id: Ie6eacb65a214d2b5a2b9a0c8f76846194f090e28
Reviewed-on: https://pigweed-review.googlesource.com/c/pigweed/kudzu/+/170857
Reviewed-by: Anthony DiGirolamo <tonymd@google.com>
Parts:
- removed JP1: GBA_SO, Jumper:SolderJumper-2_P1.3mm_Bridged_RoundedPad1.0x1.5mm
- removed JP6: GBA_SI, Jumper:SolderJumper-2_P1.3mm_Bridged_RoundedPad1.0x1.5mm
- removed JP7: GBA_SD, Jumper:SolderJumper-2_P1.3mm_Bridged_RoundedPad1.0x1.5mm
- removed JP8: GBA_SC, Jumper:SolderJumper-2_P1.3mm_Bridged_RoundedPad1.0x1.5mm
- added C29: 10nF, Capacitor_SMD:C_0603_1608Metric, F.Cu at (124.8, 39.8)
- added C30: 2.2uF, Capacitor_SMD:C_0603_1608Metric, F.Cu at (124.8, 36.9)
- added C31: 100nF, Capacitor_SMD:C_0603_1608Metric, F.Cu at (124.8, 38.3)
- added JP10: SolderJumper_3_Bridged12, Jumper:SolderJumper-3_P1.3mm_Bridged12_RoundedPad1.0x1.5mm, F.Cu at (85.5, 36.7)
- added JP11: SolderJumper_3_Bridged12, Jumper:SolderJumper-3_P1.3mm_Bridged12_RoundedPad1.0x1.5mm, F.Cu at (88.2, 36.7)
- added JP12: SolderJumper_3_Bridged12, Jumper:SolderJumper-3_P1.3mm_Bridged12_RoundedPad1.0x1.5mm, F.Cu at (90.8, 36.7)
- added JP9: SolderJumper_3_Bridged12, Jumper:SolderJumper-3_P1.3mm_Bridged12_RoundedPad1.0x1.5mm, F.Cu at (93.5, 36.7)
- added R9: 10K, Resistor_SMD:R_0603_1608Metric, F.Cu at (127.8, 49.5)
- added TP1: DISP_RESET, TestPoint:TestPoint_Pad_D1.0mm, F.Cu at (142.1, 51.1)
- added TP2: DISP_RESET, TestPoint:TestPoint_Pad_D1.0mm, F.Cu at (140.2, 49.9)
- added U3: ESP32-C3-MINI-1, Espressif:ESP32-C3-MINI-1_HandSoldering, F.Cu at (134.0, 42.3)
- moved JP5 15.1 mm to (112.3, 38.2), turned to 180 degrees
- moved TP15 3.55 mm to (132.4, 64.6)
- moved TP14 3.54 mm to (130.7, 61.5)
Connections:
- net /RP2040 and Debug/UART_RX renamed UART_RX
- net /RP2040 and Debug/UART_TX renamed UART_TX
- net /ux/TOUCH_RESET renamed TOUCH_RESET
- J7 pad 2: Net-(J7-SO) -> GBA_SO
- J7 pad 3: Net-(J7-SI) -> GBA_SI
- J7 pad 4: Net-(J7-SD) -> GBA_SD
- J7 pad 5: Net-(J7-SC) -> GBA_SC
- J9 pad 14: DISP_SDO -> /ux/DISP_SDO
- TP15 pad 1: DISP_SDO -> /ux/DISP_SDO
- U2 pad 27: DISP_SDI -> C3_RESET_N
- U2 pad 30: DISP_SDO -> DISP_SDI
- U2 pad 38: GBA_SC -> RP2040_SPI_CLK
- U2 pad 39: GBA_SO -> RP2040_SPI_DO
- U2 pad 40: GBA_SI -> RP2040_SPI_DI
- U2 pad 41: GBA_SD -> RP2040_SPI_CS
Routing:
- net DISP_SDO: track 134.6 -> 0.00 mm, vias 2 -> 0
- net RP2040_SPI_CLK: track 0.00 -> 125.9 mm
- net RP2040_SPI_DO: track 0.00 -> 125.8 mm
- net RP2040_SPI_CS: track 0.00 -> 125.8 mm
- net RP2040_SPI_DI: track 0.00 -> 125.8 mm
- net UART_RX: track 27.8 -> 147.0 mm, vias 2 -> 3
- net C3_RESET_N: track 0.00 -> 119.2 mm, vias 0 -> 2
- net UART_TX: track 25.3 -> 143.5 mm, vias 2 -> 3
- net GBA_SC: track 124.2 -> 22.8 mm, vias 0 -> 1
- net GBA_SO: track 124.1 -> 22.8 mm, vias 0 -> 1
- net GBA_SI: track 124.0 -> 22.9 mm, vias 0 -> 1
- net GBA_SD: track 124.0 -> 23.0 mm, vias 0 -> 1
- net /misc/C3_MTMS: track 0.00 -> 58.2 mm
- net /misc/C3_MTDO: track 0.00 -> 58.2 mm
- net /misc/C3_MTDI: track 0.00 -> 55.0 mm, vias 0 -> 2
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
Commit message: pcb: Rev 1
Change-Id: I2fad54877c276634b40f8b906584c28dce30efe2
Reviewed-on: https://pigweed-review.googlesource.com/c/pigweed/kudzu/+/173032
Reviewed-by: Anthony DiGirolamo <anthony.digirolamo@gmail.com>
Reviewed-by: Anthony DiGirolamo <tonymd@google.com>
Parts:
- added REF**: Fiducial_1mm_Mask2mm, Fiducial:Fiducial_1mm_Mask2mm, F.Cu at (68.0, 152.0)
- added REF**: Fiducial_1mm_Mask2mm, Fiducial:Fiducial_1mm_Mask2mm, F.Cu at (68.0, 38.0)
- added REF**: ferris, KudzuLibrary:ferris, F.Cu at (93.7, 142.3)
- added REF**: Fiducial_1mm_Mask2mm, Fiducial:Fiducial_1mm_Mask2mm, F.Cu at (142.0, 152.0)
- Q3: value Q_NMOS_DGS -> Q_NMOS_GSD
- R18, R21: value 60R 1% -> 60.4R 1%
- R24, R6: value 4K -> 4.02K 1%
- moved JP2 25.3 mm to (141.4, 83.0), turned to 90 degrees
- moved JP3 22.9 mm to (138.9, 83.0)
- moved TP8 22.8 mm to (136.7, 79.5), turned to -90 degrees
- moved C23 20.9 mm to (147.5, 75.3), turned to 180 degrees
- moved TP9 19.4 mm to (136.7, 77.5), turned to -90 degrees
- moved C22 18.5 mm to (147.5, 73.8), turned to 180 degrees
- moved C21 16.2 mm to (147.5, 72.3), turned to 180 degrees
- moved TP10 15.3 mm to (131.8, 74.7), turned to 180 degrees
- moved TP13 11.5 mm to (130.1, 71.8), turned to 180 degrees
- moved U8 11.0 mm to (132.9, 63.5), turned to 90 degrees
- moved TP12 10.2 mm to (131.8, 72.7), turned to 180 degrees
- moved TP11 10.2 mm to (130.1, 73.8), turned to 180 degrees
- moved TP14 9.27 mm to (131.8, 70.7), turned to 180 degrees
- moved JP4 7.71 mm to (136.2, 63.5), turned to -90 degrees
- moved TP15 5.66 mm to (130.1, 69.8), turned to 180 degrees
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Connections:
- J6 pad 1: UART_TX -> GND
- J6 pad 3: GND -> UART_TX
- Q3 pad 1: Net-(Q3-D) -> /power/POWER_SW_N
- Q3 pad 2: /power/POWER_SW_N -> GND
- Q3 pad 3: GND -> Net-(Q3-D)
- U2 pad 27: C3_RESET_N -> DISP_FMARK
- U2 pad 32: DISP_FMARK -> C3_RESET_N
- U8 pad 4: /ux/DISP_LEDK_2 -> /ux/DISP_LEDK_0
- U8 pad 6: /ux/DISP_LEDK_0 -> /ux/DISP_LEDK_2
Routing:
- net TOUCH_IRQ: track 140.6 -> 120.1 mm, vias 0 -> 4
- net TOUCH_RESET: track 92.8 -> 108.4 mm, vias 3 -> 5
- net SENSOR_SCL: track 127.8 -> 114.2 mm
- net /ux/DISP_IOVCC: track 11.6 -> 25.2 mm
- net /ux/DISP_VCI: track 12.1 -> 25.4 mm
- net SENSOR_SDA: track 126.7 -> 115.0 mm
- net DISP_D_C: track 137.7 -> 128.9 mm
- net GND: track 205.2 -> 212.3 mm, vias 100 -> 99
- net /ux/DISP_LEDK_2: track 8.20 -> 15.2 mm
- net /power/POWER_SW_N: track 80.4 -> 74.3 mm, vias 0 -> 2
- net /ux/DISP_LEDK_1: track 8.02 -> 14.0 mm
- net DISP_FMARK: track 137.4 -> 131.8 mm
- net /ux/DISP_LEDK_0: track 8.21 -> 12.8 mm
- net /ux/BUTTON_LEFT: track 41.7 -> 46.0 mm
- net /ux/DISP_RESET: track 75.6 -> 71.3 mm, vias 0 -> 2
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Other:
- board text added: "Kudzu Rev 1 Copyright 2023 The Pigweed Authors pigweed.dev/kudzu"
- board text removed: "Kudzu Rev 0 Copyright 2023 The Pigweed Authors pigweed.dev/kudzu"
