File: pcb/rp2040.kicad_sch (KiCad schematic)
At the start: 40 parts, among them J1 USB_C_Receptacle_USB2.0, J2 ARM 10 Pin SWD, J3 6 Pin Tag Connect, J6 Conn_01x03, U1 W25Q32JVZP, U2 RP2040, Y1 12 MHz

Commit message: pcb: Update schematic to WIP6
Change-Id: I9e9f727ad2774ee986f2f97450dc509901129aec
Reviewed-on: https://pigweed-review.googlesource.com/c/pigweed/kudzu/+/169650
Reviewed-by: Anthony DiGirolamo <tonymd@google.com>
Parts:
- J1: footprint (none) -> Connector_USB:USB_C_Receptacle_GCT_USB4105-xx-A_16P_TopMnt_Horizontal; DigiKey PN (none) -> 2073-USB4105-GF-ATR-ND; Price @ 10 (none) -> 0.68800; Price @ 25 (none) -> 0.66000
- R14, R15, R19, R20: value 2.2K -> 3.3K
- U1: DigiKey PN (none) -> W25Q128JVPIQ-ND; Price @ 10 (none) -> 1.53200; Price @ 25 (none) -> 1.49080
- U2: DigiKey PN (none) -> 2648-SC0914(13)TR-ND; Price @ 10 (none) -> 0.70; Price @ 25 (none) -> 0.70
- Y1: DigiKey PN (none) -> 2151-RH100-12.000-12-1010-EXT-TRCT-ND; Price @ 10 (none) -> 0.19500; Price @ 25 (none) -> 0.17580
Other:
- note added: "RP2040 Decaps"
- note added: "RP2040 Flash"
- note added: "TODO: Tune passives for XTAL"
- note removed: "RP2040"
- moved on the sheet: C1, C10, C11, C2, C3, C4, C5, C6, C7, C8, C9, J1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

Commit message: pcb: Update pcb to WIP7
Changes:

- Pruned unused parts from `kudzu-parts.kicad_sym`.
- Updated all parts in `kudzu-parts.kicad_sym` to pass `klc-check/check_symbol.py`.
- Switched to `PI4IOE5V6416` IO expander which has programmable pull-up.
- Removed pull-ups on `BOARD_ID*`, `BUTTON_*`, `TOUCH_RESET`, and `DISP_RESET`
  in favor of internal pull-ups in the IO expander.
- Added pull-up to `RESET_N`.
- Removed test points from `QSPI_*`.
- Switched to QFN version of `MCP73831`.
- Fixed missing pin number on `MAX17048` `QSTRT`.
- Removed pull-up on 3.3V regulator's `EN` pin and tied directly to `VIN`.
- Added extra decoupling caps to rp2040's 3.3V and 1.1V lines per design guide.
- Added note to add axis diagram to silk screen on board.
- Miscellaneous visual cleanup.
- Added FET on conduction path for system power.
- Added circuit to charge at 250mA when system is on and 500mA when system is off.
- Assigned all RP2040 IOs.
- Created and switched to dedicated symbols for DPAD, A/B, and SELECT/START.
- Switched display connector symbol for one with a mounting pin.
- Set test point values to net names.
- Selected LEDs and current limiting resistor values.
- Added closed solder jumpers to GBA Link signals.
- Changed solder jumper on GBA VCC pin to open.
- Changed LCD decoupling to mach reference circuit.
- Connected DISP_RD (J9 Pin 12) to +3V3.
- Connected DB0-15 (J9 Pins 17-32) to GND.
- Updated 12MHz Crystal (Y1) to correct symbol and foot print.

Change-Id: I6d0fe442c50df116031305f5165b6a29d3572d45
Reviewed-on: https://pigweed-review.googlesource.com/c/pigweed/kudzu/+/169858
Reviewed-by: Anthony DiGirolamo <tonymd@google.com>
Parts:
- removed TP1: QSPI_CS_N, symbol Connector:TestPoint
- removed TP2: QSPI_SD0, symbol Connector:TestPoint
- removed TP3: QSPI_SD1, symbol Connector:TestPoint
- removed TP4: QSPI_SD2, symbol Connector:TestPoint
- removed TP5: QSPI_SD3, symbol Connector:TestPoint
- removed TP6: QSPI_SCLK, symbol Connector:TestPoint
- added C11, C8: 100nF, Capacitor_SMD:C_0603_1608Metric, symbol Device:C_Small
- added R7: 10K, Resistor_SMD:R_0603_1608Metric, symbol Device:R_Small
- C1, C10, C11, C2, C3, C4, C5, C6, C7, C8, C9: footprint (none) -> Capacitor_SMD:C_0603_1608Metric
- J2: footprint (none) -> Connector_PinHeader_1.27mm:PinHeader_2x05_P1.27mm_Vertical_SMD
- J6: footprint (none) -> Connector_PinHeader_1.27mm:PinHeader_1x03_P1.27mm_Vertical_SMD_Pin1Right
- R1, R14, R15, R16, R17, R19, R2, R20, R3, R4, R5: footprint (none) -> Resistor_SMD:R_0603_1608Metric
- TP17: value RUN -> SENSOR_SCL; footprint (none) -> TestPoint:TestPoint_Pad_D1.0mm
- TP18: value RUN -> SENSOR_SDA; footprint (none) -> TestPoint:TestPoint_Pad_D1.0mm
- TP19: value RUN -> IO_SCL; footprint (none) -> TestPoint:TestPoint_Pad_D1.0mm
- TP20: value RUN -> IO_SDA; footprint (none) -> TestPoint:TestPoint_Pad_D1.0mm
- TP7: value RUN -> RESET_N; footprint (none) -> TestPoint:TestPoint_Pad_D1.0mm
- U1: value W25Q32JVZP -> W25Q128JVPIQ
- Y1: footprint (none) -> Crystal:Crystal_SMD_3225-4Pin_3.2x2.5mm; symbol Device:Crystal -> Device:Crystal_GND24_Small
Connections:
- net +1V1: now also C11.1
- net +3V3: now also C8.1, R7.2
- net GND: now also Y1.2, Y1.4, C11.2, C8.2
- net IO_SCL: now also U2.5 (GPIO3)
- net IO_SDA: now also U2.4 (GPIO2)
- net RESET_N: now also R7.1
- net SENSOR_SCL: now also U2.32 (GPIO21)
- net SENSOR_SDA: now also U2.31 (GPIO20)
- net UART_RX: now also U2.3 (GPIO1)
- net UART_TX: now also U2.2 (GPIO0)
- net at C1.2, U2.20 (XIN): now also Y1.3; no longer Y1.2
- net TOUCH_IRQ: now reaches U2.11 (GPIO8)
- net IMU_INT2: now reaches U2.12 (GPIO9)
- net IMU_FSYNC: now reaches U2.13 (GPIO10)
- net IO_INT_N: now reaches U2.14 (GPIO11)
- net IO_RESET_N: now reaches U2.15 (GPIO12)
- net DISP_BACKLIGHT: now reaches U2.16 (GPIO13)
- net DISP_FMARK: now reaches U2.17 (GPIO14)
- net DISP_D_C: now reaches U2.18 (GPIO15)
- net DISP_SDI: now reaches U2.27 (GPIO16)
- net DISP_CS_N: now reaches U2.28 (GPIO17)
- net DISP_CLK: now reaches U2.29 (GPIO18)
- net DISP_SDO: now reaches U2.30 (GPIO19)
- net AUDIO_DATA: now reaches U2.34 (GPIO22)
- net AUDIO_BCLK: now reaches U2.35 (GPIO23)
- net AUDIO_LRCLK: now reaches U2.36 (GPIO24)
- net AUDIO_SD: now reaches U2.37 (GPIO25)
- net GBA_SC: now reaches U2.38 (GPIO26_ADC0)
- net GBA_SO: now reaches U2.39 (GPIO27_ADC1)
- net GBA_SI: now reaches U2.40 (GPIO28_ADC2)
- net GBA_SD: now reaches U2.41 (GPIO29_ADC3)
- net STATUS_R: now reaches U2.6 (GPIO4)
- net STATUS_G: now reaches U2.7 (GPIO5)
- net STATUS_B: now reaches U2.8 (GPIO6)
- net GAUGE_ALERT_N: now reaches U2.9 (GPIO7)
Other:
- note added: "Pullup not needed by chosen flash part"
- note added: "RP2040"
- note removed: "Install pullup if needed by flash part."
- note removed: "TODO: Choose flash size"
- moved on the sheet: C1, C2, C3, C4, C5, C6, C7, C8, R1, R14, R15, R19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

Commit message: pcb: rev 0-r1 - board routed
Change-Id: Icb9c0ddbcf21cc7f2bac7bbcd371ff5a97baf35d
Reviewed-on: https://pigweed-review.googlesource.com/c/pigweed/kudzu/+/170233
Reviewed-by: Anthony DiGirolamo <tonymd@google.com>
Parts:
- removed C8: 100nF, Capacitor_SMD:C_0603_1608Metric, symbol Device:C_Small
- removed TP7: RESET_N, TestPoint:TestPoint_Pad_D1.0mm, symbol Connector:TestPoint
- added C8 (x2): 100nF, Capacitor_SMD:C_0603_1608Metric, symbol Device:C_Small
- added C9: 2.2uF, Capacitor_SMD:C_0603_1608Metric, symbol Device:C_Small
- C10, C9: value 1uF -> 2.2uF
- J6: footprint Connector_PinHeader_1.27mm:PinHeader_1x03_P1.27mm_Vertical_SMD_Pin1Right -> Connector_Harwin:Harwin_M20-89003xx_1x03_P2.54mm_Horizontal; DigiKey PN (none) -> 952-3264-ND; Price @ 10 (none) -> 0.47600; Price @ 25 (none) -> 0.47600
Connections:
- net +3V3: now also J2.1 (VTref), J3.1 (VCC), C8.1, C8.1, C9.1
- net AUDIO_BCLK: now also U2.8 (GPIO6); no longer U2.35 (GPIO23)
- net AUDIO_DATA: now also U2.7 (GPIO5); no longer U2.34 (GPIO22)
- net AUDIO_LRCLK: now also U2.9 (GPIO7); no longer U2.36 (GPIO24)
- net AUDIO_SD: now also U2.6 (GPIO4); no longer U2.37 (GPIO25)
- net DISP_BACKLIGHT: now also U2.18 (GPIO15); no longer U2.16 (GPIO13)
- net DISP_D_C: now also U2.31 (GPIO20); no longer U2.18 (GPIO15)
- net DISP_FMARK: now also U2.32 (GPIO21); no longer U2.17 (GPIO14)
- net GAUGE_ALERT_N: now also U2.17 (GPIO14); no longer U2.9 (GPIO7)
- net GND: now also C8.2, C8.2, C9.2
- net IMU_FSYNC: now also U2.16 (GPIO13); no longer U2.13 (GPIO10)
- net IMU_INT2: now also U2.15 (GPIO12); no longer U2.12 (GPIO9)
- net IO_RESET_N: now also U2.13 (GPIO10); no longer U2.15 (GPIO12)
- net SENSOR_SCL: now also U2.12 (GPIO9); no longer U2.32 (GPIO21)
- net SENSOR_SDA: now also U2.11 (GPIO8); no longer U2.31 (GPIO20)
- net STATUS_B: now also U2.37 (GPIO25); no longer U2.8 (GPIO6)
- net STATUS_G: now also U2.36 (GPIO24); no longer U2.7 (GPIO5)
- net STATUS_R: now also U2.35 (GPIO23); no longer U2.6 (GPIO4)
- net TOUCH_IRQ: now also U2.34 (GPIO22); no longer U2.11 (GPIO8)
- net VBUS: no longer J2.1 (VTref), J3.1 (VCC)
Other:
- company: (none) -> Copyright 2023 The Pigweed Authors
- moved on the sheet: R14, R15, TP17, TP18

Commit message: pcb: Rev 0-rc2
Change-Id: I24dc5247317789b953b5f4a603b2224101365fed
Reviewed-on: https://pigweed-review.googlesource.com/c/pigweed/kudzu/+/170855
Reviewed-by: Anthony DiGirolamo <tonymd@google.com>
Parts:
- J2: now not fitted
Connections:
- net USB_DM renamed USBD_N
- net USB_DP renamed USBD_P
Changed lines of the file:
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@@
     (title "Kudzu")
     (date "2023-09-12")
-    (rev "rev0-rc1")
+    (rev "0-rc2")
     (company "Copyright 2023 The Pigweed Authors")
   )
@@
     (effects (font (size 1.27 1.27)) (justify left bottom))
   )
-  (label "USB_DP" (at 50.8 111.76 0) (fields_autoplaced)
+  (label "USBD_P" (at 50.8 111.76 0) (fields_autoplaced)
     (effects (font (size 1.27 1.27)) (justify left bottom))
   )
-  (label "USB_DM" (at 50.8 114.3 0) (fields_autoplaced)
+  (label "USBD_N" (at 50.8 114.3 0) (fields_autoplaced)
     (effects (font (size 1.27 1.27)) (justify left bottom))
   )
@@
     (effects (font (size 1.27 1.27)) (justify left bottom))
   )
-  (label "USB_DM" (at 259.08 120.65 180) (fields_autoplaced)
+  (label "USBD_N" (at 259.08 120.65 180) (fields_autoplaced)
     (effects (font (size 1.27 1.27)) (justify right bottom))
   )
@@
     (effects (font (size 1.27 1.27)) (justify right bottom))
   )
-  (label "USB_DP" (at 259.08 123.19 180) (fields_autoplaced)
+  (label "USBD_P" (at 259.08 123.19 180) (fields_autoplaced)
     (effects (font (size 1.27 1.27)) (justify right bottom))
   )
@@
   )
   (symbol (lib_id "Connector:Conn_ARM_JTAG_SWD_10") (at 186.69 50.8 0) (unit 1)
-    (in_bom yes) (on_board yes) (dnp no)
+    (in_bom yes) (on_board yes) (dnp yes)
     (property "Reference" "J2" (at 194.31 35.56 0)
       (effects (font (size 1.27 1.27)) (justify right))

Commit message: pcb: Rev 0 ready for fab!
Change-Id: Ie6eacb65a214d2b5a2b9a0c8f76846194f090e28
Reviewed-on: https://pigweed-review.googlesource.com/c/pigweed/kudzu/+/170857
Reviewed-by: Anthony DiGirolamo <tonymd@google.com>
Connections:
- net DISP_SDO is gone; now on net DISP_SDI: U2.30 (GPIO19)
- net DISP_SDI: no longer U2.27 (GPIO16)
- net GBA_SC renamed RP2040_SPI_CLK
- net GBA_SD renamed RP2040_SPI_CS
- net GBA_SI renamed RP2040_SPI_DI
- net GBA_SO renamed RP2040_SPI_DO
- new net C3_RESET_N: U2.27 (GPIO16)
Changed lines of the file:
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@@
   (title_block
     (title "Kudzu")
-    (date "2023-09-12")
-    (rev "0-rc2")
+    (date "2023-09-13")
+    (rev "0")
     (company "Copyright 2023 The Pigweed Authors")
   )
@@
     (stroke (width 0) (type default))
   )
-  (wire (pts (xy 124.46 106.68) (xy 143.51 106.68))
+  (wire (pts (xy 124.46 106.68) (xy 130.81 106.68))
     (stroke (width 0) (type default))
   )
@@
     (stroke (width 0) (type default))
   )
-  (wire (pts (xy 124.46 104.14) (xy 143.51 104.14))
+  (wire (pts (xy 124.46 104.14) (xy 130.81 104.14))
     (stroke (width 0) (type default))
   )
@@
     (effects (font (size 3 3)) (justify left bottom))
   )
-  (label "UART_TX" (at 143.51 104.14 180) (fields_autoplaced)
-    (effects (font (size 1.27 1.27)) (justify right bottom))
-  )
   (label "QSPI_SD3" (at 54.61 59.69 180) (fields_autoplaced)
     (effects (font (size 1.27 1.27)) (justify right bottom))
@@
     (effects (font (size 1.27 1.27)) (justify right bottom))
   )
-  (label "UART_RX" (at 143.51 106.68 180) (fields_autoplaced)
-    (effects (font (size 1.27 1.27)) (justify right bottom))
-  )
   (label "UART_RX" (at 252.73 45.72 0) (fields_autoplaced)
     (effects (font (size 1.27 1.27)) (justify left bottom))
@@
     )
   )
+  (global_label "C3_RESET_N" (shape input) (at 130.81 144.78 0) (fields_autoplaced)
+    (effects (font (size 1.27 1.27)) (justify left))
+    (property "Intersheetrefs" "${INTERSHEET_REFS}" (at 145.2855 144.78 0)
+      (effects (font (size 1.27 1.27)) (justify left) hide)
+    )
+  )
   (global_label "IO_INT_N" (shape input) (at 130.81 132.08 0) (fields_autoplaced)
     (effects (font (size 1.27 1.27)) (justify left))
@@
     )
   )
-  (global_label "GBA_SC" (shape input) (at 130.81 172.72 0) (fields_autoplaced)
-    (effects (font (size 1.27 1.27)) (justify left))
-    (property "Intersheetrefs" "${INTERSHEET_REFS}" (at 140.8709 172.72 0)
-      (effects (font (size 1.27 1.27)) (justify left) hide)
-    )
-  )
-  (global_label "GBA_SD" (shape input) (at 130.81 180.34 0) (fields_autoplaced)
-    (effects (font (size 1.27 1.27)) (justify left))
-    (property "Intersheetrefs" "${INTERSHEET_REFS}" (at 140.8709 180.34 0)
+  (global_label "RP2040_SPI_CLK" (shape input) (at 130.81 172.72 0) (fields_autoplaced)
+    (effects (font (size 1.27 1.27)) (justify left))
+    (property "Intersheetrefs" "${INTERSHEET_REFS}" (at 149.7608 172.72 0)
       (effects (font (size 1.27 1.27)) (justify left) hide)
     )
@@
     )
   )
-  (global_label "GBA_SO" (shape input) (at 130.81 175.26 0) (fields_autoplaced)
-    (effects (font (size 1.27 1.27)) (justify left))
-    (property "Intersheetrefs" "${INTERSHEET_REFS}" (at 140.9314 175.26 0)
-      (effects (font (size 1.27 1.27)) (justify left) hide)
-    )
-  )
   (global_label "AUDIO_DATA" (shape input) (at 130.81 116.84 0) (fields_autoplaced)
     (effects (font (size 1.27 1.27)) (justify left))
@@
     )
   )
-  (global_label "DISP_SDI" (shape input) (at 130.81 144.78 0) (fields_autoplaced)
-    (effects (font (size 1.27 1.27)) (justify left))
-    (property "Intersheetrefs" "${INTERSHEET_REFS}" (at 142.2014 144.78 0)
+  (global_label "DISP_SDI" (shape input) (at 130.81 152.4 0) (fields_autoplaced)
+    (effects (font (size 1.27 1.27)) (justify left))
+    (property "Intersheetrefs" "${INTERSHEET_REFS}" (at 142.2014 152.4 0)
+      (effects (font (size 1.27 1.27)) (justify left) hide)
+    )
+  )
+  (global_label "RP2040_SPI_CS" (shape input) (at 130.81 180.34 0) (fields_autoplaced)
+    (effects (font (size 1.27 1.27)) (justify left))
+    (property "Intersheetrefs" "${INTERSHEET_REFS}" (at 148.6722 180.34 0)
       (effects (font (size 1.27 1.27)) (justify left) hide)
     )
@@
     (effects (font (size 1.27 1.27)) (justify left))
     (property "Intersheetrefs" "${INTERSHEET_REFS}" (at 175.7657 111.76 0)
+      (effects (font (size 1.27 1.27)) (justify left) hide)
+    )
+  )
+  (global_label "UART_RX" (shape input) (at 130.81 106.68 0) (fields_autoplaced)
+    (effects (font (size 1.27 1.27)) (justify left))
+    (property "Intersheetrefs" "${INTERSHEET_REFS}" (at 141.899 106.68 0)
       (effects (font (size 1.27 1.27)) (justify left) hide)
     )
@@
     )
   )
+  (global_label "UART_TX" (shape input) (at 130.81 104.14 0) (fields_autoplaced)
+    (effects (font (size 1.27 1.27)) (justify left))
+    (property "Intersheetrefs" "${INTERSHEET_REFS}" (at 141.5966 104.14 0)
+      (effects (font (size 1.27 1.27)) (justify left) hide)
+    )
+  )
+  (global_label "RP2040_SPI_DO" (shape input) (at 130.81 175.26 0) (fields_autoplaced)
+    (effects (font (size 1.27 1.27)) (justify left))
+    (property "Intersheetrefs" "${INTERSHEET_REFS}" (at 148.7932 175.26 0)
+      (effects (font (size 1.27 1.27)) (justify left) hide)
+    )
+  )
   (global_label "AUDIO_BCLK" (shape input) (at 130.81 119.38 0) (fields_autoplaced)
     (effects (font (size 1.27 1.27)) (justify left))
@@
     )
   )
-  (global_label "GBA_SI" (shape input) (at 130.81 177.8 0) (fields_autoplaced)
-    (effects (font (size 1.27 1.27)) (justify left))
-    (property "Intersheetrefs" "${INTERSHEET_REFS}" (at 140.2057 177.8 0)
-      (effects (font (size 1.27 1.27)) (justify left) hide)
-    )
-  )
-  (global_label "DISP_SDO" (shape input) (at 130.81 152.4 0) (fields_autoplaced)
-    (effects (font (size 1.27 1.27)) (justify left))
-    (property "Intersheetrefs" "${INTERSHEET_REFS}" (at 142.9271 152.4 0)
-      (effects (font (size 1.27 1.27)) (justify left) hide)
-    )
+  (global_label "RP2040_SPI_DI" (shape input) (at 130.81 177.8 0) (fields_autoplaced)
+    (effects (font (size 1.27 1.27)) (justify left))
+    (property "Intersheetrefs" "${INTERSHEET_REFS}" (at 148.0675 177.8 0)
+      (effects (font (size 1.27 1.27)) (justify left) hide)
+    )

Commit message: pcb: Add part numbers for passives
Change-Id: Ie1730dd2a7126b7f6f602689064a4dbf8996e7b6
Reviewed-on: https://pigweed-review.googlesource.com/c/pigweed/kudzu/+/172895
Reviewed-by: Anthony DiGirolamo <anthony.digirolamo@gmail.com>
Reviewed-by: Anthony DiGirolamo <tonymd@google.com>
Parts:
- C1, C2: DigiKey PN (none) -> 13-CC0603JPNPO9BN270CT-ND; Price @ 10 (none) -> 0.03400; Price @ 25 (none) -> 0.01880
- C10, C9: DigiKey PN (none) -> 1276-1040-2-ND; Price @ 10 (none) -> 0.03460; Price @ 25 (none) -> 0.02830
- C11, C3, C4, C5, C6, C7, C8: DigiKey PN (none) -> 1276-1000-2-ND; Price @ 10 (none) -> 0.01200; Price @ 25 (none) -> 0.00856
- R1, R7: DigiKey PN (none) -> RNCP0603FTD10K0TR-ND; Price @ 10 (none) -> 0.03240; Price @ 25 (none) -> 0.02380
- R14, R15, R19, R20: DigiKey PN (none) -> 311-3.30KHRTR-ND; Price @ 10 (none) -> 0.01800; Price @ 25 (none) -> 0.01060
- R16, R17: DigiKey PN (none) -> 311-5.10KHRTR-ND; Price @ 10 (none) -> 0.01800; Price @ 25 (none) -> 0.01060
- R2, R5: DigiKey PN (none) -> RMCF0603FT1K00TR-ND; Price @ 10 (none) -> 0.01400; Price @ 25 (none) -> 0.00860
- R3, R4: DigiKey PN (none) -> 311-27.0HRTR-ND; Price @ 10 (none) -> 0.01800; Price @ 25 (none) -> 0.01060

Commit message: pcb: Swap GND and TX on UART header
Change-Id: I73d646daeb368497cf53041f50c20bcdaad23a6c
Reviewed-on: https://pigweed-review.googlesource.com/c/pigweed/kudzu/+/173031
Reviewed-by: Anthony DiGirolamo <tonymd@google.com>
Reviewed-by: Anthony DiGirolamo <anthony.digirolamo@gmail.com>
Connections:
- net GND: now also J6.1 (Pin_1); no longer J6.3 (Pin_3)
- net UART_TX: now also J6.3 (Pin_3); no longer J6.1 (Pin_1)
Changed lines of the file:
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@@
     )
   )
-  (symbol (lib_id "Connector_Generic:Conn_01x03") (at 267.97 45.72 0) (unit 1)
-    (in_bom yes) (on_board yes) (dnp no) (fields_autoplaced)
-    (property "Reference" "J6" (at 270.51 44.45 0)
+  (symbol (lib_id "Connector_Generic:Conn_01x03") (at 267.97 45.72 0) (mirror x) (unit 1)
+    (in_bom yes) (on_board yes) (dnp no)
+    (property "Reference" "J6" (at 270.51 46.99 0)
       (effects (font (size 1.27 1.27)) (justify left))
     )
-    (property "Value" "Conn_01x03" (at 270.51 46.99 0)
+    (property "Value" "Conn_01x03" (at 270.51 44.45 0)
       (effects (font (size 1.27 1.27)) (justify left))
     )

Commit message: pcb: Rev 1
Change-Id: I2fad54877c276634b40f8b906584c28dce30efe2
Reviewed-on: https://pigweed-review.googlesource.com/c/pigweed/kudzu/+/173032
Reviewed-by: Anthony DiGirolamo <anthony.digirolamo@gmail.com>
Reviewed-by: Anthony DiGirolamo <tonymd@google.com>
Connections:
- net C3_RESET_N: now also U2.32 (GPIO21); no longer U2.27 (GPIO16)
- net DISP_FMARK: now also U2.27 (GPIO16); no longer U2.32 (GPIO21)
Changed lines of the file:
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@@
   (title_block
     (title "Kudzu")
-    (date "2023-09-13")
-    (rev "0")
+    (date "2023-09-26")
+    (rev "1")
     (company "Copyright 2023 The Pigweed Authors")
   )
@@
     )
   )
-  (global_label "C3_RESET_N" (shape input) (at 130.81 144.78 0) (fields_autoplaced)
-    (effects (font (size 1.27 1.27)) (justify left))
-    (property "Intersheetrefs" "${INTERSHEET_REFS}" (at 145.2855 144.78 0)
+  (global_label "C3_RESET_N" (shape input) (at 130.81 157.48 0) (fields_autoplaced)
+    (effects (font (size 1.27 1.27)) (justify left))
+    (property "Intersheetrefs" "${INTERSHEET_REFS}" (at 145.2855 157.48 0)
       (effects (font (size 1.27 1.27)) (justify left) hide)
     )
@@
     )
   )
-  (global_label "DISP_FMARK" (shape input) (at 130.81 157.48 0) (fields_autoplaced)
-    (effects (font (size 1.27 1.27)) (justify left))
-    (property "Intersheetrefs" "${INTERSHEET_REFS}" (at 145.2857 157.48 0)
-      (effects (font (size 1.27 1.27)) (justify left) hide)
-    )
+  (global_label "DISP_FMARK" (shape input) (at 130.81 144.78 0) (fields_autoplaced)
+    (effects (font (size 1.27 1.27)) (justify left))
+    (property "Intersheetrefs" "${INTERSHEET_REFS}" (at 145.2857 144.78 0)
+      (effects (font (size 1.27 1.27)) (justify left) hide)
+    )
