File: pcb/ux.kicad_sch (KiCad schematic)
At the start: 54 parts, among them J7 GameBoy_LinkPort, J8 Conn_01x02, J9 Conn_01x40_MountingPin, SW1 AGB_DPAD, SW2 BOOT, SW3 RESET, SW4 AGB_AB, SW5 AGB_SELECT_START, U10 PI4IOE5V6416, U5 AP2502, U7 ICM-42670-P, U9 MAX98357

Commit message: pcb: Rev 0 ready for fab!
Change-Id: Ie6eacb65a214d2b5a2b9a0c8f76846194f090e28
Reviewed-on: https://pigweed-review.googlesource.com/c/pigweed/kudzu/+/170857
Reviewed-by: Anthony DiGirolamo <tonymd@google.com>
Parts:
- removed JP1: GBA_SD, Jumper:SolderJumper-2_P1.3mm_Bridged_RoundedPad1.0x1.5mm, symbol Jumper:SolderJumper_2_Bridged
- removed JP1: GBA_SC, Jumper:SolderJumper-2_P1.3mm_Bridged_RoundedPad1.0x1.5mm, symbol Jumper:SolderJumper_2_Bridged
- removed JP1: GBA_SI, Jumper:SolderJumper-2_P1.3mm_Bridged_RoundedPad1.0x1.5mm, symbol Jumper:SolderJumper_2_Bridged
- removed JP1: GBA_SO, Jumper:SolderJumper-2_P1.3mm_Bridged_RoundedPad1.0x1.5mm, symbol Jumper:SolderJumper_2_Bridged
Connections:
- net GBA_SC: now also J7.5 (SC)
- net GBA_SD: now also J7.4 (SD)
- net GBA_SI: now also J7.3 (SI)
- net GBA_SO: now also J7.2 (SO)
Changed lines of the file:
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@@
   (title_block
     (title "Kudzu")
-    (date "2023-09-12")
-    (rev "0-rc2")
+    (date "2023-09-13")
+    (rev "0")
     (company "Copyright 2023 The Pigweed Authors")
   )
@@
   (junction (at 265.43 34.29) (diameter 0) (color 0 0 0 0)
   )
-  (junction (at 254 67.31) (diameter 0) (color 0 0 0 0)
-  )
-  (no_connect (at 248.92 125.73))
+  (no_connect (at 233.68 134.62))
   (no_connect (at 177.8 139.7))
   (no_connect (at 280.67 138.43))
@@
     (stroke (width 0) (type default))
   )
-  (wire (pts (xy 121.92 35.56) (xy 125.73 35.56))
+  (wire (pts (xy 114.3 35.56) (xy 125.73 35.56))
     (stroke (width 0) (type default))
   )
@@
     (stroke (width 0) (type default))
   )
-  (wire (pts (xy 121.92 38.1) (xy 125.73 38.1))
+  (wire (pts (xy 114.3 38.1) (xy 125.73 38.1))
     (stroke (width 0) (type default))
   )
@@
     (stroke (width 0) (type default))
   )
-  (wire (pts (xy 121.92 33.02) (xy 125.73 33.02))
+  (wire (pts (xy 114.3 33.02) (xy 125.73 33.02))
     (stroke (width 0) (type default))
   )
@@
     (stroke (width 0) (type default))
   )
-  (wire (pts (xy 238.76 67.31) (xy 254 67.31))
-    (stroke (width 0) (type default))
-  )
   (wire (pts (xy 52.07 125.73) (xy 46.99 125.73))
     (stroke (width 0) (type default))
@@
     (stroke (width 0) (type default))
   )
-  (wire (pts (xy 121.92 40.64) (xy 125.73 40.64))
+  (wire (pts (xy 114.3 40.64) (xy 125.73 40.64))
     (stroke (width 0) (type default))
   )
@@
     (effects (font (size 1.27 1.27)) (justify right bottom))
   )
-  (label "TOUCH_RESET" (at 80.01 176.53 180) (fields_autoplaced)
-    (effects (font (size 1.27 1.27)) (justify right bottom))
-  )
   (label "BUTTON_A" (at 78.74 153.67 180) (fields_autoplaced)
     (effects (font (size 1.27 1.27)) (justify right bottom))
@@
     )
   )
-  (global_label "GBA_SO" (shape input) (at 114.3 33.02 180) (fields_autoplaced)
-    (effects (font (size 1.27 1.27)) (justify right))
-    (property "Intersheetrefs" "${INTERSHEET_REFS}" (at 104.1786 33.02 0)
-      (effects (font (size 1.27 1.27)) (justify right) hide)
+  (global_label "TOUCH_RESET" (shape input) (at 80.01 176.53 0) (fields_autoplaced)
+    (effects (font (size 1.27 1.27)) (justify left))
+    (property "Intersheetrefs" "${INTERSHEET_REFS}" (at 95.937 176.53 0)
+      (effects (font (size 1.27 1.27)) (justify left) hide)
     )
   )
-  (global_label "DISP_SDO" (shape input) (at 238.76 67.31 180) (fields_autoplaced)
+  (global_label "GBA_SO" (shape input) (at 114.3 33.02 180) (fields_autoplaced)
     (effects (font (size 1.27 1.27)) (justify right))
-    (property "Intersheetrefs" "${INTERSHEET_REFS}" (at 226.6429 67.31 0)
+    (property "Intersheetrefs" "${INTERSHEET_REFS}" (at 104.1786 33.02 0)
       (effects (font (size 1.27 1.27)) (justify right) hide)
     )
@@
     )
   )
-  (symbol (lib_id "Jumper:SolderJumper_2_Bridged") (at 118.11 38.1 0) (unit 1)
-    (in_bom yes) (on_board yes) (dnp no)
-    (property "Reference" "JP1" (at 123.19 39.37 0)
-      (effects (font (size 1.27 1.27)))
-    )
-    (property "Value" "GBA_SD" (at 118.11 34.29 0)
-      (effects (font (size 1.27 1.27)) hide)
-    )
-    (property "Footprint" "Jumper:SolderJumper-2_P1.3mm_Bridged_RoundedPad1.0x1.5mm" (at 118.11 38.1 0)
-      (effects (font (size 1.27 1.27)) hide)
-    )
-    (property "Datasheet" "~" (at 118.11 38.1 0)
-      (effects (font (size 1.27 1.27)) hide)
-    )
-    (property "Price @ 10" "" (at 118.11 38.1 0)
-      (effects (font (size 1.27 1.27)) hide)
-    )
-    (property "Price @ 25" "" (at 118.11 38.1 0)
-      (effects (font (size 1.27 1.27)) hide)
-    )
-    (pin "1")
-    (pin "2")
-    (instances
-      (project "kudzu"
-        (path "/30e30bdf-50e5-46a8-92c7-0e280cceabe8"
-          (reference "JP1") (unit 1)
-        )
-        (path "/30e30bdf-50e5-46a8-92c7-0e280cceabe8/162828de-0fc8-48f2-95ca-16f35e12e8ad"
-          (reference "JP7") (unit 1)
-        )
-      )
-    )
-  )
   (symbol (lib_id "power:GND") (at 44.45 85.09 0) (unit 1)
     (in_bom yes) (on_board yes) (dnp no) (fields_autoplaced)
@@
     )
   )
-  (symbol (lib_id "Jumper:SolderJumper_2_Bridged") (at 118.11 40.64 0) (unit 1)
-    (in_bom yes) (on_board yes) (dnp no)
-    (property "Reference" "JP1" (at 123.19 41.91 0)
-      (effects (font (size 1.27 1.27)))
-    )
-    (property "Value" "GBA_SC" (at 118.11 36.83 0)
-      (effects (font (size 1.27 1.27)) hide)
-    )
-    (property "Footprint" "Jumper:SolderJumper-2_P1.3mm_Bridged_RoundedPad1.0x1.5mm" (at 118.11 40.64 0)
-      (effects (font (size 1.27 1.27)) hide)
-    )
-    (property "Datasheet" "~" (at 118.11 40.64 0)
-      (effects (font (size 1.27 1.27)) hide)
-    )
-    (property "Price @ 10" "" (at 118.11 40.64 0)
-      (effects (font (size 1.27 1.27)) hide)
-    )
-    (property "Price @ 25" "" (at 118.11 40.64 0)
-      (effects (font (size 1.27 1.27)) hide)
-    )
-    (pin "1")
-    (pin "2")
-    (instances
-      (project "kudzu"
-        (path "/30e30bdf-50e5-46a8-92c7-0e280cceabe8"
-          (reference "JP1") (unit 1)
-        )
-        (path "/30e30bdf-50e5-46a8-92c7-0e280cceabe8/162828de-0fc8-48f2-95ca-16f35e12e8ad"
-          (reference "JP8") (unit 1)
-        )
-      )
-    )
-  )
   (symbol (lib_id "power:GND") (at 49.53 186.69 0) (unit 1)
     (in_bom yes) (on_board yes) (dnp no) (fields_autoplaced)
@@
     )
   )
-  (symbol (lib_id "Jumper:SolderJumper_2_Bridged") (at 118.11 35.56 0) (unit 1)
-    (in_bom yes) (on_board yes) (dnp no)
-    (property "Reference" "JP1" (at 123.19 36.83 0)
-      (effects (font (size 1.27 1.27)))
-    )
-    (property "Value" "GBA_SI" (at 118.11 31.75 0)
-      (effects (font (size 1.27 1.27)) hide)
-    )
-    (property "Footprint" "Jumper:SolderJumper-2_P1.3mm_Bridged_RoundedPad1.0x1.5mm" (at 118.11 35.56 0)
-      (effects (font (size 1.27 1.27)) hide)
-    )
-    (property "Datasheet" "~" (at 118.11 35.56 0)
-      (effects (font (size 1.27 1.27)) hide)
-    )
-    (property "Price @ 10" "" (at 118.11 35.56 0)
-      (effects (font (size 1.27 1.27)) hide)
-    )
-    (property "Price @ 25" "" (at 118.11 35.56 0)
-      (effects (font (size 1.27 1.27)) hide)
-    )
-    (pin "1")
-    (pin "2")
-    (instances
-      (project "kudzu"
-        (path "/30e30bdf-50e5-46a8-92c7-0e280cceabe8"
-          (reference "JP1") (unit 1)
-        )
-        (path "/30e30bdf-50e5-46a8-92c7-0e280cceabe8/162828de-0fc8-48f2-95ca-16f35e12e8ad"
-          (reference "JP6") (unit 1)
-        )
-      )
-    )
-  )
   (symbol (lib_id "power:GND") (at 231.14 106.68 0) (unit 1)
     (in_bom yes) (on_board yes) (dnp no) (fields_autoplaced)
@@
         )
       )
-    )
-  )
-  (symbol (lib_id "Jumper:SolderJumper_2_Bridged") (at 118.11 33.02 0) (unit 1)
-    (in_bom yes) (on_board yes) (dnp no)
-    (property "Reference" "JP1" (at 123.19 34.29 0)
-      (effects (font (size 1.27 1.27)))
-    )
-    (property "Value" "GBA_SO" (at 118.11 29.21 0)
-      (effects (font (size 1.27 1.27)) hide)
-    )
-    (property "Footprint" "Jumper:SolderJumper-2_P1.3mm_Bridged_RoundedPad1.0x1.5mm" (at 118.11 33.02 0)
-      (effects (font (size 1.27 1.27)) hide)
-    )
-    (property "Datasheet" "~" (at 118.11 33.02 0)
-      (effects (font (size 1.27 1.27)) hide)
-    )
-    (property "Price @ 10" "" (at 118.11 33.02 0)
-      (effects (font (size 1.27 1.27)) hide)
-    )
-    (property "Price @ 25" "" (at 118.11 33.02 0)
-      (effects (font (size 1.27 1.27)) hide)
-    )
-    (pin "1")
-    (pin "2")
-    (instances
-      (project "kudzu"
-        (path "/30e30bdf-50e5-46a8-92c7-0e280cceabe8"
-          (reference "JP1") (unit 1)
-        )
-        (path "/30e30bdf-50e5-46a8-92c7-0e280cceabe8/162828de-0fc8-48f2-95ca-16f35e12e8ad"
-          (reference "JP1") (unit 1)
-        )
-      )

Commit message: pcb: Add part numbers for passives
Change-Id: Ie1730dd2a7126b7f6f602689064a4dbf8996e7b6
Reviewed-on: https://pigweed-review.googlesource.com/c/pigweed/kudzu/+/172895
Reviewed-by: Anthony DiGirolamo <anthony.digirolamo@gmail.com>
Reviewed-by: Anthony DiGirolamo <tonymd@google.com>
Parts:
- C16, C17, C18: DigiKey PN (none) -> 1276-1000-2-ND; Price @ 10 (none) -> 0.01200; Price @ 25 (none) -> 0.00856
- C16: DigiKey PN (none) -> 1276-1009-2-ND; Price @ 10 (none) -> 0.02500; Price @ 25 (none) -> 0.01340
- C16, C18: DigiKey PN (none) -> 1276-1871-2-ND; Price @ 10 (none) -> 0.10800; Price @ 25 (none) -> 0.06140
- J7: Price @ 10 2.09 -> 2.8; Price @ 25 2.09 -> 2.8
- R10, R21: DigiKey PN (none) -> 311-1.50KHRTR-ND; Price @ 10 (none) -> 0.01800; Price @ 25 (none) -> 0.01060
- R11: DigiKey PN (none) -> 311-280HRTR-ND; Price @ 10 (none) -> 0.01800; Price @ 25 (none) -> 0.01800
- R11: DigiKey PN (none) -> RNCP0603FTD10K0TR-ND; Price @ 10 (none) -> 0.03240; Price @ 25 (none) -> 0.02380
- R11: DigiKey PN (none) -> 311-634KHRTR-ND; Price @ 10 (none) -> 0.01800; Price @ 25 (none) -> 0.01800
- R12, R13: value 60R 1% -> 60.4R 1%; DigiKey PN (none) -> P60.4HTR-ND; Price @ 10 (none) -> 0.04200; Price @ 25 (none) -> 0.02340
- R13: DigiKey PN (none) -> 311-100KHRTR-ND; Price @ 10 (none) -> 0.01800; Price @ 25 (none) -> 0.01060

Commit message: pcb: Rev 1
Change-Id: I2fad54877c276634b40f8b906584c28dce30efe2
Reviewed-on: https://pigweed-review.googlesource.com/c/pigweed/kudzu/+/173032
Reviewed-by: Anthony DiGirolamo <anthony.digirolamo@gmail.com>
Reviewed-by: Anthony DiGirolamo <tonymd@google.com>
Connections:
- net DISP_LEDK_0: now also U5.4 (LED3); no longer U5.6 (LED1)
- net DISP_LEDK_2: now also U5.6 (LED1); no longer U5.4 (LED3)
Changed lines of the file:
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@@
   (title_block
     (title "Kudzu")
-    (date "2023-09-13")
-    (rev "0")
+    (date "2023-09-26")
+    (rev "1")
     (company "Copyright 2023 The Pigweed Authors")
   )
@@
     (effects (font (size 1.27 1.27)) (justify right bottom))
   )
-  (label "DISP_LEDK_2" (at 247.65 137.16 180) (fields_autoplaced)
+  (label "DISP_LEDK_2" (at 247.65 142.24 180) (fields_autoplaced)
     (effects (font (size 1.27 1.27)) (justify right bottom))
   )
@@
     (effects (font (size 1.27 1.27)) (justify right bottom))
   )
-  (label "DISP_LEDK_0" (at 247.65 142.24 180) (fields_autoplaced)
+  (label "DISP_LEDK_0" (at 247.65 137.16 180) (fields_autoplaced)
     (effects (font (size 1.27 1.27)) (justify right bottom))
   )
